Commit message: kyon full

File: source/kyon_isaac/kyon_isaac/assets/kyon.urdf (robot description, URDF)
Before this commit: robot kyon, 24 links, 23 joints
Links:
- added link dagana_1_base, mass 0.96534359; visual mesh filename=./meshes/mesh_dagana_base.stl scale=0.001 0.001 0.001
- added link dagana_1_claw, mass 0.25739835; visual mesh filename=./meshes/mesh_dagana_clamp.stl scale=0.001 0.001 0.001
- added link dagana_2_base, mass 0.96534359; visual mesh filename=./meshes/mesh_dagana_base.stl scale=0.001 0.001 0.001
- added link dagana_2_claw, mass 0.25739835; visual mesh filename=./meshes/mesh_dagana_clamp.stl scale=0.001 0.001 0.001
- added link elbow_pitch_1_link, mass 1.048477; visual mesh filename=./meshes/mesh_elbow.stl scale=0.001 0.001 0.001
- added link elbow_pitch_2_link, mass 1.048477; visual mesh filename=./meshes/mesh_elbow.stl scale=0.001 0.001 0.001
- added link shoulder_pitch_1_link, mass 2.6972599; visual mesh filename=./meshes/mesh_sh_pitch.stl scale=0.001 0.001 0.001; visual mesh filename=./meshes/mesh_sh_pitch_cover.stl scale=0.001 0.001 0.001
- added link shoulder_pitch_2_link, mass 2.6972599; visual mesh filename=./meshes/mesh_sh_pitch.stl scale=0.001 0.001 0.001; visual mesh filename=./meshes/mesh_sh_pitch_cover.stl scale=0.001 0.001 0.001
- added link shoulder_yaw_1_link, mass 0.68281255; visual mesh filename=./meshes/mesh_sh_yaw.stl scale=0.001 0.001 0.001
- added link shoulder_yaw_2_link, mass 0.68281255; visual mesh filename=./meshes/mesh_sh_yaw.stl scale=0.001 0.001 0.001
- added link wrist_pitch_1_link, mass 0.8276976; visual mesh filename=./meshes/mesh_wrist_pitch.stl scale=0.001 0.001 0.001
- added link wrist_pitch_2_link, mass 0.8276976; visual mesh filename=./meshes/mesh_wrist_pitch.stl scale=0.001 0.001 0.001
- added link wrist_yaw_1_link, mass 0.13163366; visual mesh filename=./meshes/mesh_wrist_yaw.stl scale=0.001 0.001 0.001
- added link wrist_yaw_2_link, mass 0.13163366; visual mesh filename=./meshes/mesh_wrist_yaw.stl scale=0.001 0.001 0.001
- link pelvis: geometry collision box size=0.8 0.3 0.2; visual mesh filename=./meshes/mesh_pelvis.stl scale=0.001 0.001 0.001
Joints:
- added joint dagana_1_base_joint: type fixed, parent wrist_yaw_1_link, child dagana_1_base, origin xyz=0.0 0.0 0.0 rpy=0.0 0.0 0.0
- added joint dagana_1_clamp_joint: type revolute, parent dagana_1_base, child dagana_1_claw, origin xyz=0.0361625 0.016 0.044 rpy=0.0 1.57079632679 0.0, axis 0 0 1, limit lower=-3.4056 upper=3.4056 effort=25 velocity=14
- added joint dagana_2_base_joint: type fixed, parent wrist_yaw_2_link, child dagana_2_base, origin xyz=0.0 0.0 0.0 rpy=0.0 0.0 0.0
- added joint dagana_2_clamp_joint: type revolute, parent dagana_2_base, child dagana_2_claw, origin xyz=0.0361625 0.016 0.044 rpy=0.0 1.57079632679 0.0, axis 0 0 1, limit lower=-3.3266 upper=3.3266 effort=25 velocity=14
- added joint elbow_pitch_1: type revolute, parent shoulder_pitch_1_link, child elbow_pitch_1_link, origin xyz=0.0 -0.32 0.0 rpy=0.0 0.0 0.0, axis 0 0 -1, limit lower=-3 upper=3 effort=122 velocity=4.6
- added joint elbow_pitch_2: type revolute, parent shoulder_pitch_2_link, child elbow_pitch_2_link, origin xyz=0.0 -0.32 0.0 rpy=0.0 0.0 0.0, axis 0 0 -1, limit lower=-3 upper=3 effort=122 velocity=4.6
- added joint shoulder_pitch_1: type revolute, parent shoulder_yaw_1_link, child shoulder_pitch_1_link, origin xyz=0.0 0.0 0.0735 rpy=-1.57079632679 0.0 -3.14159265358, axis 0 0 1, limit lower=-3 upper=3 effort=122 velocity=4.6
- added joint shoulder_pitch_2: type revolute, parent shoulder_yaw_2_link, child shoulder_pitch_2_link, origin xyz=0.0 0.0 0.0735 rpy=-1.57079632679 0.0 0.0, axis 0 0 1, limit lower=-3 upper=3 effort=122 velocity=4.6
- added joint shoulder_yaw_1: type revolute, parent pelvis, child shoulder_yaw_1_link, origin xyz=0.28 0.0998258 0.203238 rpy=-0.3490656 0.0 0.0, axis 0 0 -1, limit lower=-3.312 upper=3.312 effort=146 velocity=3.8
- added joint shoulder_yaw_2: type revolute, parent pelvis, child shoulder_yaw_2_link, origin xyz=0.28 -0.0998258 0.203238 rpy=0.3490656 0.0 0.0, axis 0 0 -1, limit lower=-3.3458 upper=3.3458 effort=146 velocity=3.8
- added joint wrist_pitch_1: type revolute, parent elbow_pitch_1_link, child wrist_pitch_1_link, origin xyz=0.0 -0.25 0.0 rpy=0.0 0.0 0.0, axis 0 0 -1, limit lower=-2.4056 upper=2.4056 effort=25 velocity=14
- added joint wrist_pitch_2: type revolute, parent elbow_pitch_2_link, child wrist_pitch_2_link, origin xyz=0.0 -0.25 0.0 rpy=0.0 0.0 0.0, axis 0 0 -1, limit lower=-2.3266 upper=2.3266 effort=25 velocity=14
- added joint wrist_yaw_1: type revolute, parent wrist_pitch_1_link, child wrist_yaw_1_link, origin xyz=0.0 -0.13861199999999999 0.0 rpy=1.57079632679 0.0 0.0, axis 0 0 1, limit lower=-2.4056 upper=2.4056 effort=25 velocity=14
- added joint wrist_yaw_2: type revolute, parent wrist_pitch_2_link, child wrist_yaw_2_link, origin xyz=0.0 -0.13861199999999999 0.0 rpy=1.57079632679 0.0 0.0, axis 0 0 1, limit lower=-2.3266 upper=2.3266 effort=25 velocity=14
